Commit message: Added Navigation, Map Saver

File: src/my_bot/description/gz_control.xacro (robot description, xacro)
@@ -20,10 +20,11 @@
             <frame_id>odom</frame_id>
             <child_frame_id>base_link</child_frame_id>
-            <odom_publisher_frequency>30</odom_publisher_frequency>
+            <odom_publish_frequency>30</odom_publish_frequency>
         </plugin>
-        <plugin filename="gz-sim-joint-state-publisher-system" name="gz::sim::systems::JointStatePublisher">
+<plugin filename="gz-sim-joint-state-publisher-system" name="gz::sim::systems::JointStatePublisher">
             <topic>joint_states</topic>
             <joint_name>left_wheel_joint</joint_name>
             <joint_name>right_wheel_joint</joint_name>
+            <joint_name>laser_joint</joint_name>
         </plugin>
     </gazebo>

File: src/my_bot/description/lidar.xacro (robot description, xacro)
@@ -4,5 +4,5 @@
         <parent link="chassis"/>
         <child link="laser_frame"/>
-        <origin xyz="0.1 0 0.175" rpy="0 0 0"/>
+        <origin xyz="0.1 0 0.17" rpy="0 0 0"/>
     </joint>
     <link name="laser_frame">
@@ -43,6 +43,6 @@
                 </scan>
                 <range>
-                    <min>0.3</min>
-                    <max>12</max>
+                    <min>0.1</min>
+                    <max>12.0</max>
                 </range>
             </ray>

File: src/my_bot/description/robot_core.xacro (robot description, xacro)
@@ -119,13 +119,21 @@
         </xacro:inertial_sphere>
     </link>
-    <gazebo reference="caster_wheel">
-        <visual>
-            <material>
-                <diffuse>0 0 0 1</diffuse>
-                <specular>0.1 0.1 0.1 1</specular>
-            </material>
-        </visual>
-        <mu1>0.001</mu1>
-        <mu2>0.001</mu2>
-    </gazebo>
+<gazebo reference="caster_wheel">
+    <visual>
+        <material>
+            <diffuse>0 0 0 1</diffuse>
+            <specular>0.1 0.1 0.1 1</specular>
+        </material>
+    </visual>
+    <collision>
+        <surface>
+            <friction>
+                <ode>
+                    <mu>0.001</mu>
+                    <mu2>0.001</mu2>
+                </ode>
+            </friction>
+        </surface>
+    </collision>
+</gazebo>
 </robot>

Commit message: Initial commit of ROS 2 Jazzy robot

File: src/my_bot/description/gz_control.xacro (robot description, xacro)
@@ -1,5 +1,5 @@
 <?xml version="1.0"?>
 <robot xmlns:xacro="http://www.ros.org/wiki/xacro">
-    <gazebo>
+<gazebo>
         <plugin filename="gz-sim-diff-drive-system" name="gz::sim::systems::DiffDrive">
             <left_joint>left_wheel_joint</left_joint>
@@ -11,20 +11,19 @@
             <max_angular_acceleration>2</max_angular_acceleration>
             <min_angular_acceleration>-2</min_angular_acceleration>
-            <max_linear_velocity>0.5</max_linear_velocity>
-            <min_linear_velocity>-0.5</min_linear_velocity>
-            <max_angular_velocity>1</max_angular_velocity>
-            <min_angular_velocity>-1</min_angular_velocity>
+            <max_linear_velocity>1.0</max_linear_velocity>
+            <min_linear_velocity>-1.0</min_linear_velocity>
+            <max_angular_velocity>1.0</max_angular_velocity>
+            <min_angular_velocity>-1.0</min_angular_velocity>
             <topic>cmd_vel</topic>
             <odom_topic>odom</odom_topic>
+            <odom_publisher_frequency>30</odom_publisher_frequency>
             <tf_topic>tf</tf_topic>
             <frame_id>odom</frame_id>
             <child_frame_id>base_link</child_frame_id>
-            <odom_publish_frequency>30</odom_publish_frequency>
         </plugin>
-<plugin filename="gz-sim-joint-state-publisher-system" name="gz::sim::systems::JointStatePublisher">
+        <plugin filename="gz-sim-joint-state-publisher-system" name="gz::sim::systems::JointStatePublisher">
             <topic>joint_states</topic>
             <joint_name>left_wheel_joint</joint_name>
             <joint_name>right_wheel_joint</joint_name>
-            <joint_name>laser_joint</joint_name>
         </plugin>
     </gazebo>

File: src/my_bot/description/lidar.xacro (robot description, xacro)
@@ -4,5 +4,5 @@
         <parent link="chassis"/>
         <child link="laser_frame"/>
-        <origin xyz="0.1 0 0.17" rpy="0 0 0"/>
+        <origin xyz="0.1 0 0.175" rpy="0 0 0"/>
     </joint>
     <link name="laser_frame">
@@ -24,30 +24,30 @@
         </xacro:inertial_cylinder>
     </link>
-    <gazebo reference="laser_frame">
-        <material>
-            <diffuse>1 0 0 1</diffuse>
-            <specular>0.1 0.1 0.1 1</specular>
-        </material>
-        <sensor name="laser" type="gpu_lidar">
-            <pose> 0 0 0 0 0 0 </pose>
-            <visualize>true</visualize>
-            <update_rate>10</update_rate>
-            <ray>
-                <scan>
-                    <horizontal>
-                        <samples>360</samples>
-                        <resolution>1</resolution>
-                        <min_angle>-3.14</min_angle>
-                        <max_angle>3.14</max_angle>
-                    </horizontal>
-                </scan>
-                <range>
-                    <min>0.1</min>
-                    <max>12.0</max>
-                </range>
-            </ray>
-            <topic>scan</topic>
-            <gz_frame_id>laser_frame</gz_frame_id>
+<gazebo reference="laser_frame">
+    <material>
+        <diffuse>1 0 0 1</diffuse>
+        <specular>0.1 0.1 0.1 1</specular>
+    </material>
+    <sensor name="laser" type="gpu_lidar">
+        <pose> 0 0 0 0 0 0 </pose>
+        <visualize>true</visualize>
+        <update_rate>10</update_rate>
+        <ray>
+            <scan>
+                <horizontal>
+                    <samples>360</samples>
+                    <resolution>1</resolution>
+                    <min_angle>-3.14</min_angle>
+                    <max_angle>3.14</max_angle>
+                </horizontal>
+            </scan>
+            <range>
+                <min>0.1</min>
+                <max>12.0</max>
+            </range>
+        </ray>
+        <topic>scan</topic>
+        <gz_frame_id>laser_frame</gz_frame_id>
         </sensor>
-    </gazebo>
+</gazebo>
 </robot>
